File: RGBEMP ARK Control Board/Schem and Board/ARK.brd (EAGLE design)
At the start: 40.3 x 100.3 mm, 34 parts, among them IC1 LM1117MP-3.3, J2 105450-0101, U1 SN74HCT245DWRPW, U2 CP2102N-A02-GQFN24R, U3 MMDT3904-7-F, U4 SN74HCT245DWRPW

Commit message: did some things
Parts:
- added U$9: MY_HEADER, MY_HEADER:MY_HEADER
- added X1, X10, X11, X12, X13, X14, X15, X2, X24, X3, X4, X5, X6, X7, X8, X9: TERMINAL-BLOCK-3.5MM-3-PIN-LONG-PAD, Rembrandt Electronics - Terminal Block 3-5mm v1-0:TERMINAL-BLOCK-3-PIN-3.5MM-LONG-PAD
- moved R25 138.8 mm to (12.7, 71.1), turned to 180 degrees
- moved R24 133.6 mm to (12.7, 69.7), turned to 180 degrees
- moved R23 128.3 mm to (12.7, 68.2), turned to 180 degrees
- moved R22 123.1 mm to (12.7, 66.8), turned to 180 degrees
- moved R21 117.9 mm to (12.7, 65.4), turned to 180 degrees
- moved R20 112.6 mm to (12.7, 63.9), turned to 180 degrees
- moved R19 107.4 mm to (12.7, 62.5), turned to 180 degrees
- moved R18 102.2 mm to (12.7, 61.0), turned to 180 degrees
- moved R17 73.6 mm to (54.6, 15.2), turned to 180 degrees
- moved R16 70.0 mm to (54.6, 13.7), turned to 180 degrees
- moved R15 66.6 mm to (54.6, 12.3), turned to 180 degrees
- moved R12 63.4 mm to (54.6, 10.8), turned to 180 degrees
- moved R10 60.6 mm to (54.6, 9.40), turned to 180 degrees
- moved R9 58.1 mm to (54.6, 7.96), turned to 180 degrees
- moved R8 56.0 mm to (54.6, 6.52), turned to 180 degrees
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Connections:
- new net GND_BRD: X1.3, X10.3, X11.3, X12.3, X13.3, X14.3, X15.3, X2.3, X24.3, X3.3, X4.3, X5.3, X6.3, X7.3, X8.3, X9.3
- new net HEADER_CS: U$9.P$22
- new net LEDS10_5V: U$9.P$10
- new net LEDS11_5V: U$9.P$11
- new net LEDS12_5V: U$9.P$12
- new net LEDS12_5V_BRD: X1.2, X10.2, X11.2, X12.2, X13.2, X14.2, X15.2, X2.2, X24.2, X3.2, X4.2, X5.2, X6.2, X7.2, X8.2, X9.2
- new net LEDS1_5V: U$9.P$1
- new net LEDS2_5V: U$9.P$2
- new net LEDS3_5V: U$9.P$3
- new net LEDS4_5V: U$9.P$4
- new net LEDS5_5V: U$9.P$5
- new net LEDS6_5V: U$9.P$6
- new net LEDS7_5V: U$9.P$7
- new net LEDS8_5V: U$9.P$8
- new net LEDS9_5V: U$9.P$9
- new net VDD5V_BRD: X1.1, X10.1, X11.1, X12.1, X13.1, X14.1, X15.1, X2.1, X24.1, X3.1, X4.1, X5.1, X6.1, X7.1, X8.1, X9.1
- net GND: now also U$9.P$15, U$9.P$16, U$9.P$23, U$9.P$24
- net MISO: now also U$9.P$19
- net MOSI: now also U$9.P$20
- net SCK: now also U$9.P$21
- net VDD3V3: now also U$9.P$17, U$9.P$18
- net VDD5V: now also U$9.P$13, U$9.P$14, U1.1, U4.1
Routing:
- net N$9: track 0.00 -> 118.1 mm
Other:
- board size 40.3 x 100.3 mm -> 27.2 x 118.1 mm
