File: RGBEMP ARK Control Board/Schem and Board/ARK.sch (EAGLE design)
At the start: 6 parts, among them IC1 LM1117MP-3.3

Commit message: did some things
Parts:
- added C1: 0.1uF, resistor:C-USC0402
- added C8: 1uF, EEE-FC1V1R0R:EEEFC1V1R0R
- added D2: SP0503BAHTG, SP0503BAHTG:SP0503BAHTG
- added J2: 105450-0101, 105450-0101:105450-0101
- added R10, R12, R14, R15, R16, R17, R18, R19, R20, R21, R22, R23, R24, R25, R7, R8, R9: 330, Resistor_Capacitor:RC0603JR-070RL
- added R11, R13: 12k, Resistor_Capacitor:RC0603JR-070RL
- added R4: 12k, SparkFun-Resistors:12KOHM-0603-1/10W-1%
- added U$9: MY_HEADER, MY_HEADER:MY_HEADER
- added U1, U4: SN74HCT245DWRPW, SN74HCT245DWR :SN74HCT245DWRPW
- added U2: CP2102N-A02-GQFN24R, CP2102N-A02-GQFN20R:CP2102N-A02-GQFN24R
- added U3: MMDT3904-7-F, MMDT3904:MMDT3904-7-F
- added X1, X10, X11, X12, X13, X14, X15, X2, X24, X3, X4, X5, X6, X7, X8, X9: TERMINAL-BLOCK-3.5MM-3-PIN-LONG-PAD, Rembrandt Electronics - Terminal Block 3-5mm v1-0:TERMINAL-BLOCK-3.5MM-3-PIN-LONG-PAD
Connections:
- new net D+: D2.4, J2.D1+, U2.D+
- new net D-: D2.3, J2.D1-, U2.D-
- new net DTR: R13.1, U2.DTR, U3.E2
- new net EN: U3.C1
- new net GND_BRD: X1-3.K, X10-3.K, X11-3.K, X12-3.K, X13-3.K, X14-3.K, X15-3.K, X2-3.K, X24-3.K, X3-3.K, X4-3.K, X5-3.K, X6-3.K, X7-3.K, X8-3.K, X9-3.K
- new net HEADER_CS: U$9.P$22
- new net LED3V_1: U1.A1
- new net LED3V_10: U4.A2
- new net LED3V_11: U4.A3
- new net LED3V_12: U4.A4
- new net LED3V_13: U4.A5
- new net LED3V_14: U4.A6
- new net LED3V_15: U4.A7
- new net LED3V_16: U4.A8
- new net LED3V_2: U1.A2
- new net LED3V_3: U1.A3
- new net LED3V_4: U1.A4
- new net LED3V_5: U1.A5
- new net LED3V_6: U1.A6
- new net LED3V_7: U1.A7
- new net LED3V_8: U1.A8
- new net LED3V_9: U4.A1
- new net LED5V_1: R7.2
- new net LED5V_10: R19.2
- new net LED5V_11: R20.2
- new net LED5V_12: R21.2
- new net LED5V_13: R22.2
- new net LED5V_14: R23.2
- new net LED5V_15: R24.2
- new net LED5V_16: R25.2
- new net LED5V_2: R8.2
- new net LED5V_3: R9.2
- new net LED5V_4: R10.2
- new net LED5V_5: R12.2
- new net LED5V_6: R15.2
- new net LED5V_7: R16.2
- new net LED5V_8: R17.2
- new net LED5V_9: R18.2
- new net LEDS10_5V: U$9.P$10
- new net LEDS11_5V: U$9.P$11
- new net LEDS12_5V: U$9.P$12
- new net LEDS12_5V_BRD: X1-2.K, X10-2.K, X11-2.K, X12-2.K, X13-2.K, X14-2.K, X15-2.K, X2-2.K, X24-2.K, X3-2.K, X4-2.K, X5-2.K, X6-2.K, X7-2.K, X8-2.K, X9-2.K
- new net LEDS1_5V: U$9.P$1
- new net LEDS2_5V: U$9.P$2
- new net LEDS3_5V: U$9.P$3
- new net LEDS4_5V: U$9.P$4
- new net LEDS5_5V: U$9.P$5
- new net LEDS6_5V: U$9.P$6
- new net LEDS7_5V: U$9.P$7
- new net LEDS8_5V: U$9.P$8
- new net LEDS9_5V: U$9.P$9
- new net N$11: R7.1, U1.B1
- new net N$12: R8.1, U1.B2
- new net N$13: R9.1, U1.B3
- new net N$14: R10.1, U1.B4
- new net N$15: R12.1, U1.B5
- new net N$16: R15.1, U1.B6
- new net N$17: R16.1, U1.B7
- new net N$18: R14.1, U2.TXD
- new net N$19: R17.1, U1.B8
- new net N$2: C1.1, C8.1, U2.VDD
- new net N$20: R18.1, U4.B1
- new net N$21: R19.1, U4.B2
- new net N$22: R20.1, U4.B3
- new net N$23: R21.1, U4.B4
- new net N$24: R22.1, U4.B5
- new net N$25: R23.1, U4.B6
- new net N$26: R24.1, U4.B7
- new net N$27: R25.1, U4.B8
- new net N$3: J2.D2+
- new net N$4: J2.D2-
- new net N$6: R4.2, U2.!RST
- new net N$7: R11.1, U3.B2
- new net N$8: R13.2, U3.B1
- new net RTS: R11.2, U2.RTS, U3.E1
- new net SCKI: U3.C2
- new net VDD5V_BRD: X1-1.K, X10-1.K, X11-1.K, X12-1.K, X13-1.K, X14-1.K, X15-1.K, X2-1.K, X24-1.K, X3-1.K, X4-1.K, X5-1.K, X6-1.K, X7-1.K, X8-1.K, X9-1.K
- net GND: now also C1.2, C8.2, D2.1, J2.GND1, J2.GND2, J2.GND3, J2.GND4, J2.SHIELD, U$9.P$15, U$9.P$16, U$9.P$23, U$9.P$24, U1.GND, U2.GND, U4.GND
- net MISO: now also U$9.P$19
- net MOSI: now also U$9.P$20
- net RX0: now also R14.2
- net SCK: now also U$9.P$21
- net TX0: now also U2.RXD
- net VDD3V3: now also U$9.P$17, U$9.P$18
- net VDD5V: now also R4.1, U$9.P$13, U$9.P$14, U1.DIR, U1.VCC, U4.DIR, U4.VCC
- net VDD5VUSB: now also D2.2, J2.VBUS1, J2.VBUS2, J2.VBUS3, J2.VBUS4, U2.VBUS, U2.VREGIN
